File: Projects/STM32F100C_LightBox/STM32F100C_LightBox.brd (EAGLE design)
At the start: 50 x 50 mm, 1 part

Commit message: LiteBox Project started...
Parts:
- added CN1, CN2, CN3, CN4: 1X4-3.5MM, adafruit:1X04-3.5MM
- added JP1: DHT11, pinhead-2:1X03
- added JP2: DS1820, pinhead-2:1X03
- added JP3: (no value), pinhead-2:2X04
- added R1, R10, R11, R12, R2, R3, R4, R5, R6, R7, R8, R9: 150, rc-master-smd:R1206
- added U$2, U$3, U$4, U$5, U$6, U$7: IRF7313, my-library:SO-8
- moved U$1 11.2 mm to (10.0, 5.00)
Connections:
- new net GND: U$2.1, U$2.3, U$3.1, U$3.3, U$4.1, U$4.3, U$5.1, U$5.3, U$6.1, U$6.3, U$7.1, U$7.3
- new net N$1: CN1.2, U$2.7, U$2.8
- new net N$10: R4.2, U$3.4
- new net N$11: R5.2, U$4.2
- new net N$12: CN3.2, U$5.7, U$5.8
- new net N$13: CN3.3, U$5.5, U$5.6
- new net N$14: CN3.4, U$6.7, U$6.8
- new net N$15: CN4.2, U$6.5, U$6.6
- new net N$16: CN4.3, U$7.7, U$7.8
- new net N$17: CN4.4, U$7.5, U$7.6
- new net N$18: R7.2, U$5.2
- new net N$19: R8.2, U$5.4
- new net N$2: CN1.3, U$2.5, U$2.6
- new net N$20: R9.2, U$6.2
- new net N$21: R10.2, U$6.4
- new net N$22: R11.2, U$7.2
- new net N$23: R6.2, U$4.4
- new net N$24: R12.2, U$7.4
- new net N$3: CN1.4, U$3.7, U$3.8
- new net N$4: CN2.2, U$3.5, U$3.6
- new net N$5: CN2.3, U$4.7, U$4.8
- new net N$6: CN2.4, U$4.5, U$4.6
- new net N$7: R1.2, U$2.2
- new net N$8: R2.2, U$2.4
- new net N$9: R3.2, U$3.2
- new net T1C1: R9.1, U$1.PA8
- new net T1C2: R10.1, U$1.PA9
- new net T1C3: R11.1, U$1.PA10
- new net T1C4: R12.1, U$1.PA11
- new net T2C1: R1.1, U$1.PA0
- new net T2C2: R2.1, U$1.PA1
- new net T2C3: R3.1, U$1.PA2
- new net T2C4: R4.1, U$1.PA3
- new net T3C1: R5.1, U$1.PA6
- new net T3C2: R6.1, U$1.PA7
- new net T3C3: JP1.2, R7.1
- new net T3C4: JP2.2, R8.1
- net +12V: now also CN1.1, CN2.1, CN3.1, CN4.1
Other:
- board size 50 x 50 mm -> 90 x 60 mm

Commit message: LiteBox Project update...
Parts:
- added JP4: TSOPxx36, pinhead-2:1X03
- moved JP3 80.5 mm to (76.2, 33.7), turned to 270 degrees
- moved CN2 72.3 mm to (10.0, 27.5), turned to 0 degrees
- moved CN4 70.7 mm to (10.0, 52.5)
- moved CN3 70.1 mm to (10.0, 40.0)
- moved CN1 69.6 mm to (10.0, 15.0), turned to 0 degrees
- moved U$7 46.5 mm to (24.8, 52.6), turned to 180 degrees
- moved U$4 44.9 mm to (24.6, 28.9), turned to 180 degrees
- moved U$2 41.2 mm to (24.5, 12.0), turned to 180 degrees
- moved U$6 41.2 mm to (24.8, 44.9), turned to 180 degrees
- moved U$5 41.0 mm to (24.6, 37.4), turned to 180 degrees
- moved U$3 40.3 mm to (24.6, 20.8), turned to 180 degrees
- moved R7 34.2 mm to (34.2, 30.6), turned to 180 degrees
- moved R6 26.6 mm to (40.1, 25.7), turned to 180 degrees
- moved R12 26.1 mm to (40.6, 53.1), turned to 180 degrees
- moved R5 25.4 mm to (33.9, 22.4), turned to 180 degrees
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Connections:
- new net PA15: JP3.3
- new net PB3: JP3.6
- new net PB4: JP3.8
- new net PB5: JP3.5
- new net PB7: JP3.7
- new net T4C1: JP3.4, JP4.1
- new net VDD: JP3.1, JP4.3
- net GND: now also JP3.2, JP4.2
Routing:
- net GND: track 0.00 -> 142.6 mm
- net T3C3: track 0.00 -> 61.0 mm
- net T3C1: track 0.00 -> 45.7 mm
- net T3C4: track 0.00 -> 39.6 mm
- net +12V: track 0.00 -> 37.5 mm
- net T1C1: track 0.00 -> 35.4 mm
- net T3C2: track 0.00 -> 31.6 mm
- net T1C3: track 0.00 -> 26.9 mm
- net T1C2: track 0.00 -> 26.1 mm
- net T2C3: track 0.00 -> 21.0 mm
- net N$15: track 0.00 -> 20.9 mm
- net N$4: track 0.00 -> 19.8 mm
- net T2C1: track 0.00 -> 19.2 mm
- net T2C4: track 0.00 -> 18.6 mm
- net N$1: track 0.00 -> 18.4 mm
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
Commit message: LB Audio in...
Parts:
- added JP5: (no value), my-library:AUB-13
- added R13: 1k, rc-master-smd:R1206
- moved CN1 8.60 mm to (10.0, 6.40), turned to 180 degrees
- moved CN2 8.50 mm to (6.20, 19.9), turned to 90 degrees
- moved CN3 4.74 mm to (6.10, 37.3), turned to 90 degrees
Connections:
- net GND: now also JP5.1
Routing:
- net GND: track 142.6 -> 0.00 mm
- net T3C3: track 61.0 -> 0.00 mm
- net T3C1: track 45.7 -> 0.00 mm
- net T3C4: track 39.6 -> 0.00 mm
- net +12V: track 37.5 -> 0.00 mm
- net T1C1: track 35.4 -> 0.00 mm
- net T3C2: track 31.6 -> 0.00 mm
- net T1C3: track 26.9 -> 0.00 mm
- net T1C2: track 26.1 -> 0.00 mm
- net T2C3: track 21.0 -> 0.00 mm
- net N$15: track 20.9 -> 0.00 mm
- net N$4: track 19.8 -> 0.00 mm
- net T2C1: track 19.2 -> 0.00 mm
- net T2C4: track 18.6 -> 0.00 mm
- net N$1: track 18.4 -> 0.00 mm
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
Commit message: LB Audio in...
Parts:
- added C1, C3, C6, C8: 1u, rc-master-smd:C0603
- added C10, C2, C5, C7: 100u, rc-master-smd:C0603
- added C4, C9: 200u, rc-master-smd:C0603
- added IC1, IC2: TL062D, linear:SO08
- added R14, R20: 51k, rc-master-smd:R1206
- added R15, R21: 100k, rc-master-smd:R1206
- added R16, R19, R22: 1k, rc-master-smd:R1206
- added R17, R18, R23, R24: 1.5k, rc-master-smd:R1206
- moved R13 83.2 mm to (83.2, 15.6), turned to 90 degrees
Connections:
- new net +3V3: IC1.8, IC2.8
- new net N$25: JP5.3, R13.1
- new net N$26: C1.1, R13.2
- new net N$27: C1.2, IC1.3, R14.2
- new net N$28: C2.1, IC1.2, R15.1, R16.1
- new net N$29: C2.2, IC1.1, R15.2, R17.1
- new net N$30: C3.2, R16.2
- new net N$31: JP5.2, R19.1
- new net N$32: C5.2, IC2.2, R18.2
- new net N$33: C4.1, R17.2, R18.1
- new net N$34: C4.2, IC2.1, IC2.3
- new net N$35: C6.1, R19.2
- new net N$36: C6.2, IC1.5, R20.2
- new net N$37: C7.1, IC1.6, R21.1, R22.1
- new net N$38: C7.2, IC1.7, R21.2, R23.1
- new net N$39: C8.2, R22.2
- new net N$40: C9.1, R23.2, R24.1
- new net N$41: C10.2, IC2.6, R24.2
- new net N$42: C9.2, IC2.5, IC2.7
- net GND: now also C10.1, C3.1, C5.1, C8.1, IC1.4, IC2.4, R14.1, R20.1
