File: Projects/STM32F100C_LightBox/STM32F100C_LightBox.sch (EAGLE design)
At the start: 1 part

Commit message: LiteBox Project started...
Parts:
- added CN1, CN2, CN3, CN4: 1X4-3.5MM, adafruit:1X4-3.5MM
- added JP1: DHT11, pinhead-2:PINHD-1X03_2.54
- added JP2: DS1820, pinhead-2:PINHD-1X03_2.54
- added JP3: (no value), pinhead-2:PINHD-2X04_2.54
- added R1, R10, R11, R12, R2, R3, R4, R5, R6, R7, R8, R9: 150, rc-master-smd:R_1206
- added U$2, U$3, U$4, U$5, U$6, U$7: IRF7313, my-library:IRF7313
Connections:
- new net +12V: CN1.1, CN2.1, CN3.1, CN4.1
- new net GND: U$2G$1.S, U$2G$2.S, U$3G$1.S, U$3G$2.S, U$4G$1.S, U$4G$2.S, U$5G$1.S, U$5G$2.S, U$6G$1.S, U$6G$2.S, U$7G$1.S, U$7G$2.S
- new net N$1: CN1.2, U$2G$1.D
- new net N$10: R4.2, U$3G$2.G
- new net N$11: R5.2, U$4G$1.G
- new net N$12: CN3.2, U$5G$1.D
- new net N$13: CN3.3, U$5G$2.D
- new net N$14: CN3.4, U$6G$1.D
- new net N$15: CN4.2, U$6G$2.D
- new net N$16: CN4.3, U$7G$1.D
- new net N$17: CN4.4, U$7G$2.D
- new net N$18: R7.2, U$5G$1.G
- new net N$19: R8.2, U$5G$2.G
- new net N$2: CN1.3, U$2G$2.D
- new net N$20: R9.2, U$6G$1.G
- new net N$21: R10.2, U$6G$2.G
- new net N$22: R11.2, U$7G$1.G
- new net N$23: R6.2, U$4G$2.G
- new net N$24: R12.2, U$7G$2.G
- new net N$3: CN1.4, U$3G$1.D
- new net N$4: CN2.2, U$3G$2.D
- new net N$5: CN2.3, U$4G$1.D
- new net N$6: CN2.4, U$4G$2.D
- new net N$7: R1.2, U$2G$1.G
- new net N$8: R2.2, U$2G$2.G
- new net N$9: R3.2, U$3G$1.G
- new net T1C1: R9.1, U$1.PA8
- new net T1C2: R10.1, U$1.PA9
- new net T1C3: R11.1, U$1.PA10
- new net T1C4: R12.1, U$1.PA11
- new net T2C1: R1.1, U$1.PA0
- new net T2C2: R2.1, U$1.PA1
- new net T2C3: R3.1, U$1.PA2
- new net T2C4: R4.1, U$1.PA3
- new net T3C1: R5.1, U$1.PA6
- new net T3C2: R6.1, U$1.PA7
- new net T3C3: JP1.2, R7.1
- new net T3C4: JP2.2, R8.1

Commit message: LiteBox Project update...
Parts:
- added JP4: TSOPxx36, pinhead-2:PINHD-1X03_2.54
Connections:
- new net PA15: JP3.3
- new net PB3: JP3.6
- new net PB4: JP3.8
- new net PB5: JP3.5
- new net PB7: JP3.7
- new net T4C1: JP3.4, JP4.1
- new net VDD: JP3.1, JP4.3
- net GND: now also JP3.2, JP4.2
Changed lines of the file:
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@@
 <part name="JP2" library="pinhead-2" deviceset="PINHD-1X03" device="_2.54" value="DS1820"/>
 <part name="JP3" library="pinhead-2" deviceset="PINHD-2X04" device="_2.54"/>
+<part name="JP4" library="pinhead-2" deviceset="PINHD-1X03" device="_2.54" value="TSOPxx36"/>
 </parts>
 <sheets>
@@
 <instance part="JP2" gate="A" x="63.5" y="12.7"/>
 <instance part="JP3" gate="A" x="55.88" y="-12.7"/>
+<instance part="JP4" gate="A" x="33.02" y="-10.16"/>
 </instances>
 <busses>
@@
 <pinref part="GND12" gate="1" pin="GND"/>
 </segment>
+<segment>
+<pinref part="JP4" gate="A" pin="2"/>
+<wire x1="30.48" y1="-10.16" x2="17.78" y2="-10.16" width="0.1524" layer="91"/>
+<label x="17.78" y="-10.16" size="1.778" layer="95"/>
+</segment>
+<segment>
+<pinref part="JP3" gate="A" pin="2"/>
+<wire x1="60.96" y1="-7.62" x2="71.12" y2="-7.62" width="0.1524" layer="91"/>
+<label x="66.04" y="-7.62" size="1.778" layer="95"/>
+</segment>
 </net>
 <net name="N$12" class="0">
@@
 </segment>
 </net>
+<net name="T4C1" class="0">
+<segment>
+<pinref part="JP4" gate="A" pin="1"/>
+<wire x1="30.48" y1="-7.62" x2="17.78" y2="-7.62" width="0.1524" layer="91"/>
+<label x="17.78" y="-7.62" size="1.778" layer="95"/>
+</segment>
+<segment>
+<pinref part="JP3" gate="A" pin="4"/>
+<wire x1="60.96" y1="-10.16" x2="71.12" y2="-10.16" width="0.1524" layer="91"/>
+<label x="66.04" y="-10.16" size="1.778" layer="95"/>
+</segment>
+</net>
+<net name="VDD" class="0">
+<segment>
+<pinref part="JP4" gate="A" pin="3"/>
+<wire x1="30.48" y1="-12.7" x2="17.78" y2="-12.7" width="0.1524" layer="91"/>
+<label x="17.78" y="-12.7" size="1.778" layer="95"/>
+</segment>
+<segment>
+<pinref part="JP3" gate="A" pin="1"/>
+<wire x1="53.34" y1="-7.62" x2="43.18" y2="-7.62" width="0.1524" layer="91"/>
+<label x="43.18" y="-7.62" size="1.778" layer="95"/>
+</segment>
+</net>
+<net name="PA15" class="0">
+<segment>
+<pinref part="JP3" gate="A" pin="3"/>
+<wire x1="53.34" y1="-10.16" x2="43.18" y2="-10.16" width="0.1524" layer="91"/>
+<label x="43.18" y="-10.16" size="1.778" layer="95"/>
+</segment>
+</net>
+<net name="PB3" class="0">
+<segment>
+<pinref part="JP3" gate="A" pin="6"/>
+<wire x1="60.96" y1="-12.7" x2="71.12" y2="-12.7" width="0.1524" layer="91"/>
+<label x="66.04" y="-12.7" size="1.778" layer="95"/>
+</segment>
+</net>
+<net name="PB5" class="0">
+<segment>
+<pinref part="JP3" gate="A" pin="5"/>
+<wire x1="53.34" y1="-12.7" x2="43.18" y2="-12.7" width="0.1524" layer="91"/>
+<label x="43.18" y="-12.7" size="1.778" layer="95"/>
+</segment>
+</net>
+<net name="PB7" class="0">
+<segment>
+<pinref part="JP3" gate="A" pin="7"/>
+<wire x1="53.34" y1="-15.24" x2="43.18" y2="-15.24" width="0.1524" layer="91"/>
+<label x="43.18" y="-15.24" size="1.778" layer="95"/>
+</segment>
+</net>
+<net name="PB4" class="0">
+<segment>
+<pinref part="JP3" gate="A" pin="8"/>
+<wire x1="60.96" y1="-15.24" x2="71.12" y2="-15.24" width="0.1524" layer="91"/>
+<label x="66.04" y="-15.24" size="1.778" layer="95"/>
+</segment>
+</net>

Commit message: LB Audio in...
Parts:
- added JP5: (no value), my-library:AUDIO-JACK
- added R13: 1k, rc-master-smd:R_1206
Connections:
- net GND: now also JP5.SLEEVE
Changed lines of the file:
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@@
 <grid distance="0.1" unitdist="inch" unit="inch" style="lines" multiple="1" display="no" altdistance="0.01" altunitdist="inch" altunit="inch"/>
 <layers>
-<layer number="1" name="Top" color="4" fill="1" visible="no" active="no"/>
-<layer number="16" name="Bottom" color="1" fill="1" visible="no" active="no"/>
-<layer number="17" name="Pads" color="2" fill="1" visible="no" active="no"/>
-<layer number="18" name="Vias" color="2" fill="1" visible="no" active="no"/>
-<layer number="19" name="Unrouted" color="6" fill="1" visible="no" active="no"/>
-<layer number="20" name="Dimension" color="15" fill="1" visible="no" active="no"/>
-<layer number="21" name="tPlace" color="7" fill="1" visible="no" active="no"/>
-<layer number="22" name="bPlace" color="7" fill="1" visible="no" active="no"/>
-<layer number="23" name="tOrigins" color="15" fill="1" visible="no" active="no"/>
-<layer number="24" name="bOrigins" color="15" fill="1" visible="no" active="no"/>
-<layer number="25" name="tNames" color="7" fill="1" visible="no" active="no"/>
-<layer number="26" name="bNames" color="7" fill="1" visible="no" active="no"/>
-<layer number="27" name="tValues" color="7" fill="1" visible="no" active="no"/>
-<layer number="28" name="bValues" color="7" fill="1" visible="no" active="no"/>
+<layer number="1" name="Top" color="4" fill="1" visible="yes" active="no"/>
+<layer number="16" name="Bottom" color="1" fill="1" visible="yes" active="no"/>
+<layer number="17" name="Pads" color="2" fill="1" visible="yes" active="no"/>
+<layer number="18" name="Vias" color="2" fill="1" visible="yes" active="no"/>
+<layer number="19" name="Unrouted" color="6" fill="1" visible="yes" active="no"/>
+<layer number="20" name="Dimension" color="15" fill="1" visible="yes" active="no"/>
+<layer number="21" name="tPlace" color="7" fill="1" visible="yes" active="no"/>
+<layer number="22" name="bPlace" color="7" fill="1" visible="yes" active="no"/>
+<layer number="23" name="tOrigins" color="15" fill="1" visible="yes" active="no"/>
+<layer number="24" name="bOrigins" color="15" fill="1" visible="yes" active="no"/>
+<layer number="25" name="tNames" color="7" fill="1" visible="yes" active="no"/>
+<layer number="26" name="bNames" color="7" fill="1" visible="yes" active="no"/>
+<layer number="27" name="tValues" color="7" fill="1" visible="yes" active="no"/>
+<layer number="28" name="bValues" color="7" fill="1" visible="yes" active="no"/>
 <layer number="29" name="tStop" color="7" fill="3" visible="no" active="no"/>
 <layer number="30" name="bStop" color="7" fill="6" visible="no" active="no"/>
@@
 <layer number="35" name="tGlue" color="7" fill="4" visible="no" active="no"/>
 <layer number="36" name="bGlue" color="7" fill="5" visible="no" active="no"/>
-<layer number="37" name="tTest" color="7" fill="1" visible="no" active="no"/>
-<layer number="38" name="bTest" color="7" fill="1" visible="no" active="no"/>
+<layer number="37" name="tTest" color="7" fill="1" visible="yes" active="no"/>
+<layer number="38" name="bTest" color="7" fill="1" visible="yes" active="no"/>
 <layer number="39" name="tKeepout" color="4" fill="11" visible="no" active="no"/>
 <layer number="40" name="bKeepout" color="1" fill="11" visible="no" active="no"/>
@@
 <layer number="44" name="Drills" color="7" fill="1" visible="no" active="no"/>
 <layer number="45" name="Holes" color="7" fill="1" visible="no" active="no"/>
-<layer number="46" name="Milling" color="3" fill="1" visible="no" active="no"/>
-<layer number="47" name="Measures" color="7" fill="1" visible="no" active="no"/>
-<layer number="48" name="Document" color="7" fill="1" visible="no" active="no"/>
-<layer number="49" name="Reference" color="7" fill="1" visible="no" active="no"/>
-<layer number="50" name="dxf" color="7" fill="1" visible="no" active="no"/>
-<layer number="51" name="tDocu" color="7" fill="1" visible="no" active="no"/>
-<layer number="52" name="bDocu" color="7" fill="1" visible="no" active="no"/>
-<layer number="53" name="tGND_GNDA" color="7" fill="9" visible="no" active="no"/>
-<layer number="54" name="bGND_GNDA" color="1" fill="9" visible="no" active="no"/>
-<layer number="56" name="wert" color="7" fill="1" visible="no" active="no"/>
-<layer number="57" name="tCAD" color="7" fill="1" visible="no" active="no"/>
+<layer number="46" name="Milling" color="3" fill="1" visible="yes" active="no"/>
+<layer number="47" name="Measures" color="7" fill="1" visible="yes" active="no"/>
+<layer number="48" name="Document" color="7" fill="1" visible="yes" active="no"/>
+<layer number="49" name="Reference" color="7" fill="1" visible="yes" active="no"/>
+<layer number="50" name="dxf" color="7" fill="1" visible="yes" active="no"/>
+<layer number="51" name="tDocu" color="7" fill="1" visible="yes" active="no"/>
+<layer number="52" name="bDocu" color="7" fill="1" visible="yes" active="no"/>
+<layer number="53" name="tGND_GNDA" color="7" fill="9" visible="yes" active="no"/>
+<layer number="54" name="bGND_GNDA" color="1" fill="9" visible="yes" active="no"/>
+<layer number="56" name="wert" color="7" fill="1" visible="yes" active="no"/>
+<layer number="57" name="tCAD" color="7" fill="1" visible="yes" active="no"/>
 <layer number="90" name="Modules" color="5" fill="1" visible="yes" active="yes"/>
 <layer number="91" name="Nets" color="2" fill="1" visible="yes" active="yes"/>
@@
 <part name="JP3" library="pinhead-2" deviceset="PINHD-2X04" device="_2.54"/>
 <part name="JP4" library="pinhead-2" deviceset="PINHD-1X03" device="_2.54" value="TSOPxx36"/>
+<part name="JP5" library="my-library" deviceset="AUDIO-JACK" device=""/>
+<part name="GND13" library="supply1" deviceset="GND" device=""/>
+<part name="R13" library="rc-master-smd" deviceset="R_" device="1206" value="1k"/>
 </parts>
 <sheets>
@@
 <instance part="JP3" gate="A" x="55.88" y="-12.7"/>
 <instance part="JP4" gate="A" x="33.02" y="-10.16"/>
+<instance part="JP5" gate="G$1" x="22.86" y="-38.1" rot="MR180"/>
+<instance part="GND13" gate="1" x="27.94" y="-45.72"/>
+<instance part="R13" gate="G$1" x="48.26" y="-35.56"/>
 </instances>
 <busses>
@@
 <label x="66.04" y="-7.62" size="1.778" layer="95"/>
 </segment>
-</net>
+<segment>
+<pinref part="JP5" gate="G$1" pin="SLEEVE"/>
+<pinref part="GND13" gate="1" pin="GND"/>
+<wire x1="27.94" y1="-40.64" x2="27.94" y2="-43.18" width="0.1524" layer="91"/>
+</segment>
+</net>

Commit message: LB Audio in...
Parts:
- added C1, C3, C6, C8: 1u, rc-master-smd:C_0603
- added C10, C2, C5, C7: 100u, rc-master-smd:C_0603
- added C4, C9: 200u, rc-master-smd:C_0603
- added IC1, IC2: TL062D, linear:TL062D
- added R14, R20: 51k, rc-master-smd:R_1206
- added R15, R21: 100k, rc-master-smd:R_1206
- added R16, R19, R22: 1k, rc-master-smd:R_1206
- added R17, R18, R23, R24: 1.5k, rc-master-smd:R_1206
Connections:
- new net +3V3: IC1P.V+, IC2P.V+
- new net N$25: JP5.LEFT, R13.1
- new net N$26: C1.1, R13.2
- new net N$27: C1.2, IC1A.+IN, R14.2
- new net N$28: C2.1, IC1A.-IN, R15.1, R16.1
- new net N$29: C2.2, IC1A.OUT, R15.2, R17.1
- new net N$30: C3.2, R16.2
- new net N$31: JP5.RIGHT, R19.1
- new net N$32: C5.2, IC2A.-IN, R18.2
- new net N$33: C4.1, R17.2, R18.1
- new net N$34: C4.2, IC2A.+IN, IC2A.OUT
- new net N$35: C6.1, R19.2
- new net N$36: C6.2, IC1B.+IN, R20.2
- new net N$37: C7.1, IC1B.-IN, R21.1, R22.1
- new net N$38: C7.2, IC1B.OUT, R21.2, R23.1
- new net N$39: C8.2, R22.2
- new net N$40: C9.1, R23.2, R24.1
- new net N$41: C10.2, IC2B.-IN, R24.2
- new net N$42: C9.2, IC2B.+IN, IC2B.OUT
- net GND: now also C10.1, C3.1, C5.1, C8.1, IC1P.V-, IC2P.V-, R14.1, R20.1
